Commit message: added new urdf in simviz

File: models/panda_arm_gripper.urdf (robot description, URDF)
Before this commit: robot panda_arm_gripper, 11 links, 10 joints
Links:
- removed link end-effector
- added link force-sensor, mass 0.255; visual cylinder length=0.0375 radius=0.0375; visual mesh filename=meshes/visual/hand.obj
- link link7: mass 1.8 -> 0.627143; geometry visual mesh filename=meshes/visual/link7.obj
Joints:
- removed joint joint_ee
- added joint joint_force_sensor: type fixed, parent link7, child force-sensor, origin xyz=0 0 0.12 rpy=0 0 0
- joint finger_joint1: origin xyz=0 0 0.1654 rpy=0 0 -0.78539816339 -> xyz=0 0 0.21 rpy=0 0 -0.78539816339
- joint finger_joint2: origin xyz=0 0 0.1654 rpy=0 0 2.35619449019 -> xyz=0 0 0.21 rpy=0 0 2.35619449019
